Commit message: Add explicit Fortress and Harmonic simulation support

File: urdf/chassis.urdf.xacro (robot description, xacro)
@@ -2,72 +2,166 @@
 <!-- SPDX-License-Identifier: Apache-2.0 -->
 <robot xmlns:xacro="http://www.ros.org/wiki/xacro">
-  <!-- Physical links, joints, limits and inertias. Gazebo systems live in plugins. -->
+  <!-- Physical links, joints, limits and inertias. -->
   <xacro:macro name="swerve_chassis" params="prefix geometry control">
-    <xacro:property name="wheelbase" value="${geometry['wheelbase']}"/>
-    <xacro:property name="track_width" value="${geometry['track_width']}"/>
-    <xacro:property name="wheel_radius" value="${geometry['wheel_radius']}"/>
-    <xacro:property name="wheel_width" value="${geometry['wheel_width']}"/>
-    <xacro:property name="body_length" value="${geometry['body_length']}"/>
-    <xacro:property name="body_width" value="${geometry['body_width']}"/>
-    <xacro:property name="body_height" value="${geometry['body_height']}"/>
-    <xacro:property name="ground_clearance" value="${geometry['ground_clearance']}"/>
-    <xacro:property name="body_mass" value="${geometry['body_mass']}"/>
-    <xacro:property name="wheel_mass" value="${geometry['wheel_mass']}"/>
-    <xacro:property name="steering_mass" value="${geometry['steering_mass']}"/>
-    <xacro:property name="steering_limit" value="${control['steering_limit']}"/>
-    <xacro:property name="max_wheel_speed" value="${control['max_wheel_speed']}"/>
-    <xacro:property name="max_steering_rate" value="${control['max_steering_rate']}"/>
-    <xacro:property name="base_z" value="${ground_clearance + body_height / 2}"/>
-    <material name="body_blue"><color rgba="0.12 0.35 0.65 1"/></material>
-    <material name="rubber"><color rgba="0.12 0.12 0.14 1"/></material>
-    <material name="steer_orange"><color rgba="1.0 0.45 0.08 1"/></material>
-    <link name="${prefix}base_footprint"/>
+    <xacro:property name="wheelbase" value="${geometry['wheelbase']}" />
+    <xacro:property name="track_width" value="${geometry['track_width']}" />
+    <xacro:property name="wheel_radius" value="${geometry['wheel_radius']}" />
+    <xacro:property name="wheel_width" value="${geometry['wheel_width']}" />
+    <xacro:property name="body_length" value="${geometry['body_length']}" />
+    <xacro:property name="body_width" value="${geometry['body_width']}" />
+    <xacro:property name="body_height" value="${geometry['body_height']}" />
+    <xacro:property
+      name="ground_clearance"
+      value="${geometry['ground_clearance']}"
+    />
+    <xacro:property name="body_mass" value="${geometry['body_mass']}" />
+    <xacro:property name="wheel_mass" value="${geometry['wheel_mass']}" />
+    <xacro:property
+      name="steering_mass"
+      value="${geometry['steering_mass']}"
+    />
+    <xacro:property
+      name="steering_limit"
+      value="${control['steering_limit']}"
+    />
+    <xacro:property
+      name="max_wheel_speed"
+      value="${control['max_wheel_speed']}"
+    />
+    <xacro:property
+      name="max_steering_rate"
+      value="${control['max_steering_rate']}"
+    />
+    <xacro:property
+      name="base_z"
+      value="${ground_clearance + body_height / 2}"
+    />
+    <material name="body_blue">
+      <color rgba="0.12 0.35 0.65 1" />
+    </material>
+    <material name="rubber">
+      <color rgba="0.12 0.12 0.14 1" />
+    </material>
+    <material name="steer_orange">
+      <color rgba="1.0 0.45 0.08 1" />
+    </material>
+    <link name="${prefix}base_footprint" />
     <joint name="${prefix}base_joint" type="fixed">
-      <parent link="${prefix}base_footprint"/><child link="${prefix}base_link"/>
-      <origin xyz="0 0 ${base_z}"/>
+      <parent link="${prefix}base_footprint" />
+      <child link="${prefix}base_link" />
+      <origin xyz="0 0 ${base_z}" />
     </joint>
     <link name="${prefix}base_link">
-      <visual><geometry><box size="${body_length} ${body_width} ${body_height}"/></geometry><material name="body_blue"/></visual>
-      <collision><geometry><box size="${body_length} ${body_width} ${body_height}"/></geometry></collision>
+      <visual>
+        <geometry>
+          <box size="${body_length} ${body_width} ${body_height}" />
+        </geometry>
+        <material name="body_blue" />
+      </visual>
+      <collision>
+        <geometry>
+          <box size="${body_length} ${body_width} ${body_height}" />
+        </geometry>
+      </collision>
       <inertial>
-        <mass value="${body_mass}"/>
-        <inertia ixx="${body_mass*(body_width*body_width+body_height*body_height)/12}" iyy="${body_mass*(body_length*body_length+body_height*body_height)/12}"
-                 izz="${body_mass*(body_length*body_length+body_width*body_width)/12}" ixy="0" ixz="0" iyz="0"/>
+        <mass value="${body_mass}" />
+        <inertia
+          ixx="${body_mass * (body_width * body_width + body_height * body_height) / 12}"
+          ixy="0"
+          ixz="0"
+          iyy="${body_mass * (body_length * body_length + body_height * body_height) / 12}"
+          iyz="0"
+          izz="${body_mass * (body_length * body_length + body_width * body_width) / 12}"
+        />
       </inertial>
     </link>
     <xacro:macro name="swerve_module" params="name x y">
       <joint name="${prefix}${name}_steering_joint" type="revolute">
-        <parent link="${prefix}base_link"/><child link="${prefix}${name}_steering_link"/>
-        <origin xyz="${x} ${y} ${wheel_radius-base_z}"/>
-        <axis xyz="0 0 1"/>
-        <limit lower="${-steering_limit}" upper="${steering_limit}"
-               effort="30" velocity="${max_steering_rate}"/>
-        <dynamics damping="0.1" friction="0.0"/>
+        <parent link="${prefix}base_link" />
+        <child link="${prefix}${name}_steering_link" />
+        <origin xyz="${x} ${y} ${wheel_radius - base_z}" />
+        <axis xyz="0 0 1" />
+        <limit
+          lower="${-steering_limit}"
+          upper="${steering_limit}"
+          effort="30"
+          velocity="${max_steering_rate}"
+        />
+        <dynamics damping="0.1" friction="0.0" />
       </joint>
       <link name="${prefix}${name}_steering_link">
-        <visual><origin xyz="0 0 ${wheel_radius*0.65}"/><geometry><box size="0.04 0.04 0.04"/></geometry><material name="steer_orange"/></visual>
-        <inertial><mass value="${steering_mass}"/>
-          <inertia ixx="${steering_mass*0.04*0.04/6}" iyy="${steering_mass*0.04*0.04/6}" izz="${steering_mass*0.04*0.04/6}" ixy="0" ixz="0" iyz="0"/>
+        <visual>
+          <origin xyz="0 0 ${wheel_radius * 0.65}" />
+          <geometry>
+            <box size="0.04 0.04 0.04" />
+          </geometry>
+          <material name="steer_orange" />
+        </visual>
+        <inertial>
+          <mass value="${steering_mass}" />
+          <inertia
+            ixx="${steering_mass * 0.04 * 0.04 / 6}"
+            ixy="0"
+            ixz="0"
+            iyy="${steering_mass * 0.04 * 0.04 / 6}"
+            iyz="0"
+            izz="${steering_mass * 0.04 * 0.04 / 6}"
+          />
         </inertial>
       </link>
       <joint name="${prefix}${name}_wheel_joint" type="continuous">
-        <parent link="${prefix}${name}_steering_link"/><child link="${prefix}${name}_wheel_link"/>
-        <axis xyz="0 1 0"/>
-        <limit effort="20" velocity="${max_wheel_speed}"/>
-        <dynamics damping="0.01" friction="0.0"/>
+        <parent link="${prefix}${name}_steering_link" />
+        <child link="${prefix}${name}_wheel_link" />
+        <axis xyz="0 1 0" />
+        <limit effort="20" velocity="${max_wheel_speed}" />
+        <dynamics damping="0.01" friction="0.0" />
       </joint>
       <link name="${prefix}${name}_wheel_link">
-        <visual><origin rpy="${pi/2} 0 0"/><geometry><cylinder radius="${wheel_radius}" length="${wheel_width}"/></geometry><material name="rubber"/></visual>
-        <collision><origin rpy="${pi/2} 0 0"/><geometry><cylinder radius="${wheel_radius}" length="${wheel_width}"/></geometry></collision>
-        <inertial><mass value="${wheel_mass}"/>
-          <inertia ixx="${wheel_mass*(3*wheel_radius*wheel_radius+wheel_width*wheel_width)/12}" iyy="${wheel_mass*wheel_radius*wheel_radius/2}"
-                   izz="${wheel_mass*(3*wheel_radius*wheel_radius+wheel_width*wheel_width)/12}" ixy="0" ixz="0" iyz="0"/>
+        <visual>
+          <origin rpy="${pi / 2} 0 0" />
+          <geometry>
+            <cylinder radius="${wheel_radius}" length="${wheel_width}" />
+          </geometry>
+          <material name="rubber" />
+        </visual>
+        <collision>
+          <origin rpy="${pi / 2} 0 0" />
+          <geometry>
+            <cylinder radius="${wheel_radius}" length="${wheel_width}" />
+          </geometry>
+        </collision>
+        <inertial>
+          <mass value="${wheel_mass}" />
+          <inertia
+            ixx="${wheel_mass * (3 * wheel_radius * wheel_radius + wheel_width * wheel_width) / 12}"
+            ixy="0"
+            ixz="0"
+            iyy="${wheel_mass * wheel_radius * wheel_radius / 2}"
+            iyz="0"
+            izz="${wheel_mass * (3 * wheel_radius * wheel_radius + wheel_width * wheel_width) / 12}"
+          />
         </inertial>
       </link>
     </xacro:macro>
-    <xacro:swerve_module name="fl" x="${wheelbase/2}" y="${track_width/2}"/>
-    <xacro:swerve_module name="fr" x="${wheelbase/2}" y="${-track_width/2}"/>
-    <xacro:swerve_module name="rl" x="${-wheelbase/2}" y="${track_width/2}"/>
-    <xacro:swerve_module name="rr" x="${-wheelbase/2}" y="${-track_width/2}"/>
+    <xacro:swerve_module
+      name="fl"
+      x="${wheelbase / 2}"
+      y="${track_width / 2}"
+    />
+    <xacro:swerve_module
+      name="fr"
+      x="${wheelbase / 2}"
+      y="${-track_width / 2}"
+    />
+    <xacro:swerve_module
+      name="rl"
+      x="${-wheelbase / 2}"
+      y="${track_width / 2}"
+    />
+    <xacro:swerve_module
+      name="rr"
+      x="${-wheelbase / 2}"
+      y="${-track_width / 2}"
+    />
   </xacro:macro>
 </robot>

File: urdf/plugins.urdf.xacro (robot description, xacro)
@@ -2,47 +2,100 @@
 <!-- SPDX-License-Identifier: Apache-2.0 -->
 <robot xmlns:xacro="http://www.ros.org/wiki/xacro">
-  <!-- Gazebo contact and systems are kept separate from the chassis links. -->
-  <xacro:macro name="swerve_plugins" params="prefix namespace controllers_file control publish_ground_truth robot_name">
-    <xacro:property name="max_wheel_speed" value="${control['max_wheel_speed']}"/>
-    <xacro:property name="steering_limit" value="${control['steering_limit']}"/>
+  <!-- Gazebo contact, ros2_control and validation plugins. -->
+  <xacro:macro
+    name="swerve_plugins"
+    params="prefix namespace controllers_file control publish_ground_truth gazebo_version"
+  >
+    <xacro:property
+      name="max_wheel_speed"
+      value="${control['max_wheel_speed']}"
+    />
+    <xacro:property
+      name="steering_limit"
+      value="${control['steering_limit']}"
+    />
+    <xacro:property
+      name="ground_truth_topic"
+      value="${namespace + '/ground_truth/odom' if namespace else '/ground_truth/odom'}"
+    />
     <xacro:macro name="wheel_contact" params="corner">
-      <gazebo reference="${prefix}${corner}_wheel_link"><mu1>1.0</mu1><mu2>1.0</mu2></gazebo>
+      <gazebo reference="${prefix}${corner}_wheel_link">
+        <mu1>1.0</mu1>
+        <mu2>1.0</mu2>
+      </gazebo>
     </xacro:macro>
-    <xacro:wheel_contact corner="fl"/>
-    <xacro:wheel_contact corner="fr"/>
-    <xacro:wheel_contact corner="rl"/>
-    <xacro:wheel_contact corner="rr"/>
+    <xacro:wheel_contact corner="fl" />
+    <xacro:wheel_contact corner="fr" />
+    <xacro:wheel_contact corner="rl" />
+    <xacro:wheel_contact corner="rr" />
     <xacro:macro name="control_module" params="name">
       <joint name="${prefix}${name}_wheel_joint">
-        <command_interface name="velocity"><param name="min">${-max_wheel_speed}</param><param name="max">${max_wheel_speed}</param></command_interface>
-        <state_interface name="position"/><state_interface name="velocity"/>
+        <command_interface name="velocity">
+          <param name="min">${-max_wheel_speed}</param>
+          <param name="max">${max_wheel_speed}</param>
+        </command_interface>
+        <state_interface name="position" />
+        <state_interface name="velocity" />
       </joint>
       <joint name="${prefix}${name}_steering_joint">
-        <command_interface name="position"><param name="min">${-steering_limit}</param><param name="max">${steering_limit}</param></command_interface>
-        <state_interface name="position"/><state_interface name="velocity"/>
+        <command_interface name="position">
+          <param name="min">${-steering_limit}</param>
+          <param name="max">${steering_limit}</param>
+        </command_interface>
+        <state_interface name="position" />
+        <state_interface name="velocity" />
       </joint>
     </xacro:macro>
     <ros2_control name="${prefix}SwerveSystem" type="system">
-      <hardware><plugin>gz_ros2_control/GazeboSimSystem</plugin></hardware>
-      <xacro:control_module name="fl"/><xacro:control_module name="fr"/>
-      <xacro:control_module name="rl"/><xacro:control_module name="rr"/>
+      <hardware>
+        <plugin>gz_ros2_control/GazeboSimSystem</plugin>
+      </hardware>
+      <xacro:control_module name="fl" />
+      <xacro:control_module name="fr" />
+      <xacro:control_module name="rl" />
+      <xacro:control_module name="rr" />
     </ros2_control>
     <gazebo>
-      <plugin filename="gz_ros2_control-system" name="gz_ros2_control::GazeboSimROS2ControlPlugin">
+      <plugin
+        filename="gz_ros2_control-system"
+        name="gz_ros2_control::GazeboSimROS2ControlPlugin"
+      >
         <parameters>${controllers_file}</parameters>
         <robot_param>robot_description</robot_param>
-        <!-- gz_ros2_control prepends its own ROS namespace to this node name. -->
         <robot_param_node>robot_state_publisher</robot_param_node>
-        <ros><namespace>${namespace if namespace else '/'}</namespace></ros>
+        <ros>
+          <namespace>${namespace if namespace else '/'}</namespace>
+        </ros>
       </plugin>
     </gazebo>
     <xacro:if value="${publish_ground_truth}">
-      <gazebo>
-        <plugin filename="ignition-gazebo-odometry-publisher-system" name="ignition::gazebo::systems::OdometryPublisher">
-          <odom_frame>${prefix}world</odom_frame><robot_base_frame>${prefix}base_footprint</robot_base_frame>
-          <odom_publish_frequency>50</odom_publish_frequency><dimensions>2</dimensions>
-          <odom_topic>/model/${robot_name}/odometry</odom_topic>
-        </plugin>
-      </gazebo>
+      <xacro:if value="${gazebo_version == 'ign'}">
+        <gazebo>
+          <plugin
+            filename="ignition-gazebo-odometry-publisher-system"
+            name="ignition::gazebo::systems::OdometryPublisher"
+          >
+            <odom_frame>${prefix}world</odom_frame>
+            <robot_base_frame>${prefix}base_footprint</robot_base_frame>
+            <odom_publish_frequency>50</odom_publish_frequency>
+            <dimensions>2</dimensions>
+            <odom_topic>${ground_truth_topic}</odom_topic>
+          </plugin>
+        </gazebo>
+      </xacro:if>
+      <xacro:if value="${gazebo_version == 'gz'}">
+        <gazebo>
+          <plugin
+            filename="gz-sim-odometry-publisher-system"
+            name="gz::sim::systems::OdometryPublisher"
+          >
+            <odom_frame>${prefix}world</odom_frame>
+            <robot_base_frame>${prefix}base_footprint</robot_base_frame>
+            <odom_publish_frequency>50</odom_publish_frequency>
+            <dimensions>2</dimensions>
+            <odom_topic>${ground_truth_topic}</odom_topic>
+          </plugin>
+        </gazebo>
+      </xacro:if>
     </xacro:if>
   </xacro:macro>

File: urdf/swerve_drive.urdf.xacro (robot description, xacro)
@@ -3,16 +3,28 @@
 <robot xmlns:xacro="http://www.ros.org/wiki/xacro" name="swerve_drive">
   <!-- Public simulation model: chassis geometry plus Gazebo plugins. -->
-  <xacro:arg name="config_file" default="$(find swerve_gazebo_sim)/config/swerve.yaml"/>
-  <xacro:arg name="prefix" default=""/>
-  <xacro:arg name="namespace" default=""/>
-  <xacro:arg name="controllers_file" default=""/>
-  <xacro:arg name="publish_ground_truth" default="false"/>
-  <xacro:arg name="robot_name" default="swerve"/>
-  <xacro:property name="settings" value="${xacro.load_yaml('$(arg config_file)')}"/>
-  <xacro:include filename="$(find swerve_gazebo_sim)/urdf/chassis.urdf.xacro"/>
-  <xacro:include filename="$(find swerve_gazebo_sim)/urdf/plugins.urdf.xacro"/>
-  <xacro:swerve_chassis prefix="$(arg prefix)"
-                        geometry="${settings['geometry']}"
-                        control="${settings['control']}"/>
+  <xacro:arg
+    name="config_file"
+    default="$(find swerve_gazebo_sim)/config/swerve.yaml"
+  />
+  <xacro:arg name="gazebo_version" default="ign" />
+  <xacro:arg name="prefix" default="" />
+  <xacro:arg name="namespace" default="" />
+  <xacro:arg name="controllers_file" default="" />
+  <xacro:arg name="publish_ground_truth" default="false" />
+  <xacro:property
+    name="settings"
+    value="${xacro.load_yaml('$(arg config_file)')}"
+  />
+  <xacro:include
+    filename="$(find swerve_gazebo_sim)/urdf/chassis.urdf.xacro"
+  />
+  <xacro:include
+    filename="$(find swerve_gazebo_sim)/urdf/plugins.urdf.xacro"
+  />
+  <xacro:swerve_chassis
+    prefix="$(arg prefix)"
+    geometry="${settings['geometry']}"
+    control="${settings['control']}"
+  />
   <xacro:swerve_plugins
     prefix="$(arg prefix)"
@@ -21,4 +33,5 @@
     control="${settings['control']}"
     publish_ground_truth="$(arg publish_ground_truth)"
-    robot_name="$(arg robot_name)"/>
+    gazebo_version="$(arg gazebo_version)"
+  />
 </robot>
